Commit message: 260113-调整了一部分USD模型的问题

File: source/moudle/pipe_robot/urdf/pipe_robot.urdf (robot description, URDF)
Before this commit: robot pipe_robot, 53 links, 52 joints
Links:
- link BL_05_link: geometry collision mesh filename=package://pipe_robot/meshes/BL_05_link.STL; visual mesh filename=package://pipe_robot/meshes/BL_05_link.STL
- link BL_05_link_copy1: geometry collision mesh filename=package://pipe_robot/meshes/BL_05_link_copy1.STL; visual mesh filename=package://pipe_robot/meshes/BL_05_link_copy1.STL
- link BL_05_link_copy2: geometry collision mesh filename=package://pipe_robot/meshes/BL_05_link_copy2.STL; visual mesh filename=package://pipe_robot/meshes/BL_05_link_copy2.STL
- link BL_10_link: geometry collision mesh filename=package://pipe_robot/meshes/BL_10_link.STL; visual mesh filename=package://pipe_robot/meshes/BL_10_link.STL
- link BL_12_link: geometry collision mesh filename=package://pipe_robot/meshes/BL_12_link.STL; visual mesh filename=package://pipe_robot/meshes/BL_12_link.STL
- link BL_14_link: geometry collision mesh filename=package://pipe_robot/meshes/BL_14_link.STL; visual mesh filename=package://pipe_robot/meshes/BL_14_link.STL
- link BL_16_link: geometry collision mesh filename=package://pipe_robot/meshes/BL_16_link.STL; visual mesh filename=package://pipe_robot/meshes/BL_16_link.STL
- link BL_18_link: geometry collision mesh filename=package://pipe_robot/meshes/BL_18_link.STL; visual mesh filename=package://pipe_robot/meshes/BL_18_link.STL
- link BL_20_link: geometry collision mesh filename=package://pipe_robot/meshes/BL_20_link.STL; visual mesh filename=package://pipe_robot/meshes/BL_20_link.STL
- link BL_22_link: geometry collision mesh filename=package://pipe_robot/meshes/BL_22_link.STL; visual mesh filename=package://pipe_robot/meshes/BL_22_link.STL
- link BM_01_link: geometry collision mesh filename=package://pipe_robot/meshes/BM_01_link.STL; visual mesh filename=package://pipe_robot/meshes/BM_01_link.STL
- link BM_02_link_cam: geometry collision mesh filename=package://pipe_robot/meshes/BM_02_link_cam.STL; visual mesh filename=package://pipe_robot/meshes/BM_02_link_cam.STL
- link BM_03_link_imu: geometry collision mesh filename=package://pipe_robot/meshes/BM_03_link_imu.STL; visual mesh filename=package://pipe_robot/meshes/BM_03_link_imu.STL
- link BM_04_link: geometry collision mesh filename=package://pipe_robot/meshes/BM_04_link.STL; visual mesh filename=package://pipe_robot/meshes/BM_04_link.STL
- link BM_07_link: geometry collision mesh filename=package://pipe_robot/meshes/BM_07_link.STL; visual mesh filename=package://pipe_robot/meshes/BM_07_link.STL
- link BM_08_link: geometry collision mesh filename=package://pipe_robot/meshes/BM_08_link.STL; visual mesh filename=package://pipe_robot/meshes/BM_08_link.STL
- link BM_09_link: geometry collision mesh filename=package://pipe_robot/meshes/BM_09_link.STL; visual mesh filename=package://pipe_robot/meshes/BM_09_link.STL
- link BR_06_link: geometry collision mesh filename=package://pipe_robot/meshes/BR_06_link.STL; visual mesh filename=package://pipe_robot/meshes/BR_06_link.STL
- link BR_06_link_copy1: geometry collision mesh filename=package://pipe_robot/meshes/BR_06_link_copy1.STL; visual mesh filename=package://pipe_robot/meshes/BR_06_link_copy1.STL
- link BR_06_link_copy2: geometry collision mesh filename=package://pipe_robot/meshes/BR_06_link_copy2.STL; visual mesh filename=package://pipe_robot/meshes/BR_06_link_copy2.STL
- link BR_11_link: geometry collision mesh filename=package://pipe_robot/meshes/BR_11_link.STL; visual mesh filename=package://pipe_robot/meshes/BR_11_link.STL
- link BR_13_link: geometry collision mesh filename=package://pipe_robot/meshes/BR_13_link.STL; visual mesh filename=package://pipe_robot/meshes/BR_13_link.STL
- link BR_15_link: geometry collision mesh filename=package://pipe_robot/meshes/BR_15_link.STL; visual mesh filename=package://pipe_robot/meshes/BR_15_link.STL
- link BR_17_link: geometry collision mesh filename=package://pipe_robot/meshes/BR_17_link.STL; visual mesh filename=package://pipe_robot/meshes/BR_17_link.STL
- link BR_19_link: geometry collision mesh filename=package://pipe_robot/meshes/BR_19_link.STL; visual mesh filename=package://pipe_robot/meshes/BR_19_link.STL
- link BR_21_link: geometry collision mesh filename=package://pipe_robot/meshes/BR_21_link.STL; visual mesh filename=package://pipe_robot/meshes/BR_21_link.STL
- link BR_23_link: geometry collision mesh filename=package://pipe_robot/meshes/BR_23_link.STL; visual mesh filename=package://pipe_robot/meshes/BR_23_link.STL
- link FL_28_link: geometry collision mesh filename=package://pipe_robot/meshes/FL_28_link.STL; visual mesh filename=package://pipe_robot/meshes/FL_28_link.STL
- link FL_28_link_copy1: geometry collision mesh filename=package://pipe_robot/meshes/FL_28_link_copy1.STL; visual mesh filename=package://pipe_robot/meshes/FL_28_link_copy1.STL
- link FL_28_link_copy2: geometry collision mesh filename=package://pipe_robot/meshes/FL_28_link_copy2.STL; visual mesh filename=package://pipe_robot/meshes/FL_28_link_copy2.STL
- link FL_32_link: geometry collision mesh filename=package://pipe_robot/meshes/FL_32_link.STL; visual mesh filename=package://pipe_robot/meshes/FL_32_link.STL
- link FL_34_link: geometry collision mesh filename=package://pipe_robot/meshes/FL_34_link.STL; visual mesh filename=package://pipe_robot/meshes/FL_34_link.STL
- link FL_36_link: geometry collision mesh filename=package://pipe_robot/meshes/FL_36_link.STL; visual mesh filename=package://pipe_robot/meshes/FL_36_link.STL
- link FL_38_link: geometry collision mesh filename=package://pipe_robot/meshes/FL_38_link.STL; visual mesh filename=package://pipe_robot/meshes/FL_38_link.STL
- link FL_40_link: geometry collision mesh filename=package://pipe_robot/meshes/FL_40_link.STL; visual mesh filename=package://pipe_robot/meshes/FL_40_link.STL
- link FL_42_link: geometry collision mesh filename=package://pipe_robot/meshes/FL_42_link.STL; visual mesh filename=package://pipe_robot/meshes/FL_42_link.STL
- link FL_44_link: geometry collision mesh filename=package://pipe_robot/meshes/FL_44_link.STL; visual mesh filename=package://pipe_robot/meshes/FL_44_link.STL
- link FL_45_link: geometry collision mesh filename=package://pipe_robot/meshes/FL_45_link.STL; visual mesh filename=package://pipe_robot/meshes/FL_45_link.STL
- link FM_24_link: geometry collision mesh filename=package://pipe_robot/meshes/FM_24_link.STL; visual mesh filename=package://pipe_robot/meshes/FM_24_link.STL
- link FM_25_link_cam: geometry collision mesh filename=package://pipe_robot/meshes/FM_25_link_cam.STL; visual mesh filename=package://pipe_robot/meshes/FM_25_link_cam.STL
- link FM_26_link_imu: geometry collision mesh filename=package://pipe_robot/meshes/FM_26_link_imu.STL; visual mesh filename=package://pipe_robot/meshes/FM_26_link_imu.STL
- link FM_27_link: geometry collision mesh filename=package://pipe_robot/meshes/FM_27_link.STL; visual mesh filename=package://pipe_robot/meshes/FM_27_link.STL
- link FM_30_link: geometry collision mesh filename=package://pipe_robot/meshes/FM_30_link.STL; visual mesh filename=package://pipe_robot/meshes/FM_30_link.STL
- link FM_31_link: geometry collision mesh filename=package://pipe_robot/meshes/FM_31_link.STL; visual mesh filename=package://pipe_robot/meshes/FM_31_link.STL
- link FR_29_link: geometry collision mesh filename=package://pipe_robot/meshes/FR_29_link.STL; visual mesh filename=package://pipe_robot/meshes/FR_29_link.STL
- link FR_29_link_copy1: geometry collision mesh filename=package://pipe_robot/meshes/FR_29_link_copy1.STL; visual mesh filename=package://pipe_robot/meshes/FR_29_link_copy1.STL
- link FR_29_link_copy2: geometry collision mesh filename=package://pipe_robot/meshes/FR_29_link_copy2.STL; visual mesh filename=package://pipe_robot/meshes/FR_29_link_copy2.STL
- link FR_33_link: geometry collision mesh filename=package://pipe_robot/meshes/FR_33_link.STL; visual mesh filename=package://pipe_robot/meshes/FR_33_link.STL
- link FR_35_link: geometry collision mesh filename=package://pipe_robot/meshes/FR_35_link.STL; visual mesh filename=package://pipe_robot/meshes/FR_35_link.STL
- link FR_37_link: geometry collision mesh filename=package://pipe_robot/meshes/FR_37_link.STL; visual mesh filename=package://pipe_robot/meshes/FR_37_link.STL
- link FR_39_link: geometry collision mesh filename=package://pipe_robot/meshes/FR_39_link.STL; visual mesh filename=package://pipe_robot/meshes/FR_39_link.STL
- link FR_41_link: geometry collision mesh filename=package://pipe_robot/meshes/FR_41_link.STL; visual mesh filename=package://pipe_robot/meshes/FR_41_link.STL
- link FR_43_link: geometry collision mesh filename=package://pipe_robot/meshes/FR_43_link.STL; visual mesh filename=package://pipe_robot/meshes/FR_43_link.STL
Joints:
- joint joint_01_04_LF: axis 0 0 -1 -> 0 0 1; limit lower=0 upper=0 effort=0 velocity=0 -> lower=-0.0385 upper=0.015 effort=0 velocity=0
- joint joint_01_07_RF: axis 0 0 -1 -> 0 0 1
- joint joint_01_09_RF: axis 0 0 -1 -> 0 0 1; limit (none) -> lower=-0.488692 upper=1.047197533 effort=600 velocity=0.5; type continuous -> revolute
- joint joint_04_10_RN: origin xyz=0.0002000000000002 0.138 0.0455144934992005 rpy=3.14159265358979 -1.5707963267949 0 -> xyz=0.0002000000000002 0.138 0.0455144934992005 rpy=0 -1.5707963267949 0
- joint joint_04_11_RN: origin xyz=-0.000199999999999756 -0.138 0.0455144934992005 rpy=3.14159265358979 -1.5707963267949 0 -> xyz=-0.000199999999999756 -0.138 0.0455144934992005 rpy=0.0 -1.5707963267949 0
- joint joint_05_14_RF: limit (none) -> lower=-0.488692 upper=1.274090 effort=600 velocity=0.8; type continuous -> revolute
- joint joint_06_15_RF: limit (none) -> lower=-0.488692 upper=1.274090 effort=600 velocity=0.8; type continuous -> revolute
- joint joint_07_08_RF: origin xyz=0 0 0.019 rpy=3.14159265358979 -1.5707963267949 0 -> xyz=0 0 0.019 rpy=3.14159265358979 1.5707963267949 0
- joint joint_09_24_RF: limit (none) -> lower=-0.488692 upper=1.047197533 effort=600 velocity=0.5; type continuous -> revolute
- joint joint_10_12_LF: axis 0 0 -1 -> 0 0 1; limit lower=0 upper=0 effort=0 velocity=0 -> lower=-0.011 upper=0 effort=360 velocity=0.06
- joint joint_11_13_LF: axis 0 0 -1 -> 0 0 1; limit lower=0 upper=0 effort=0 velocity=0 -> lower=-0.011 upper=0 effort=360 velocity=0.06
- joint joint_16_20_RF: axis 0 0 -1 -> 0 0 1
- joint joint_17_21_RF: axis 0 0 -1 -> 0 0 1
- joint joint_21_23_RF: axis 0 0 -1 -> 0 0 1
- joint joint_24_27_LF: axis 0 0 -1 -> 0 0 1; limit lower=0 upper=0 effort=0 velocity=0 -> lower=-0.0385 upper=0.015 effort=3000 velocity=0.05
- joint joint_24_30_RF: origin xyz=0.084 0.062 -0.07 rpy=3.1416 -1.5708 0 -> xyz=0.084 0.062 -0.07 rpy=3.1416 -1.5708 3.14159
- joint joint_27_32_RN: origin xyz=0.0001999999999997 0.138 0.0455144934992005 rpy=0 -1.5707963267949 0 -> xyz=0.0001999999999997 0.138 0.0455144934992005 rpy=3.14159 -1.5707963267949 0
- joint joint_28_36_RF: limit (none) -> lower=-0.488692 upper=1.274090 effort=600 velocity=0.8; type continuous -> revolute
- joint joint_29_37_RF: limit (none) -> lower=-0.488692 upper=1.274090 effort=600 velocity=0.8; type continuous -> revolute
- joint joint_30_31_RF: axis 0 0 -1 -> 0 0 1; origin xyz=0 0 0.019 rpy=3.1416 -1.5708 0 -> xyz=0 0 0.019 rpy=3.1416 1.5708 0
- joint joint_32_34_LF: axis 0 0 -1 -> 0 0 1; limit lower=0 upper=0 effort=0 velocity=0 -> lower=-0.011 upper=0 effort=360 velocity=0.06
- joint joint_33_35_LF: axis 0 0 -1 -> 0 0 1; limit lower=0 upper=0 effort=0 velocity=0 -> lower=-0.011 upper=0 effort=360 velocity=0.06
- joint joint_38_42_RF: axis 0 0 -1 -> 0 0 1
- joint joint_39_43_RF: axis 0 0 -1 -> 0 0 1
- joint joint_42_44_RF: axis 0 0 -1 -> 0 0 1
